File: NOR/NOR.kicad_pcb (KiCad board)
At the start: 2 copper layers, 0 parts

Commit message: Finish NOR gate PCB and unify NAND with it
Parts:
- added D1: Green, LED_SMD:LED_0603_1608Metric, F.Cu at (132.3, 87.2)
- added J1: 5-146280-3-ND, Logic:PinHeader_1x03_P2.54mm_Vertical_Top, B.Cu at (127.0, 76.2)
- added J2: 5-146280-3-ND, Logic:PinHeader_1x03_P2.54mm_Vertical_Bottom, B.Cu at (127.0, 94.0)
- added Q1: DMP2004K-7, Package_TO_SOT_SMD:SOT-23, F.Cu at (129.4, 83.7)
- added Q2: DMP2004K-7, Package_TO_SOT_SMD:SOT-23, F.Cu at (129.4, 87.6)
- added R1: 10k, Resistor_SMD:R_0603_1608Metric, F.Cu at (129.4, 90.4)
- added R2: 150, Resistor_SMD:R_0603_1608Metric, F.Cu at (132.3, 84.1)
Routing:
- net /Y: track 0.00 -> 14.7 mm
- net /B: track 0.00 -> 11.2 mm
- net GND: track 0.00 -> 7.89 mm
- net VDC: track 0.00 -> 7.16 mm
- net /A: track 0.00 -> 6.90 mm
- net Net-(Q1-D): track 0.00 -> 2.86 mm
- net Net-(D1-A): track 0.00 -> 1.56 mm
Other:
- board outline added: 7.9 x 20.6 mm
- board text added: "A"
- board text added: "B"
- board text added: "GND"
- board text added: "NOR"
- board text added: "VDC"
- board text added: "Y"
- board text added: "Y=~{A+B}"
